Commit message: Initial upload of diff robot URDF + ros2_control

File: src/botlab_diff_description/botlab_diff_description/urdf/diff_drive_car.urdf.xacro (robot description, xacro)
@@ -2,9 +2,9 @@
 <robot name="diff_car" xmlns:xacro="http://www.ros.org/wiki/xacro">
   <!-- 参数 -->
-  <xacro:property name="wheel_radius" value="0.03"/>
-  <xacro:property name="wheel_width"  value="0.02"/>
-  <xacro:property name="base_length"  value="0.20"/>
-  <xacro:property name="base_width"   value="0.15"/>
-  <xacro:property name="base_height"  value="0.05"/>
+  <xacro:property name="wheel_radius" value="0.035"/>
+  <xacro:property name="wheel_width"  value="0.025"/>
+  <xacro:property name="base_length"  value="0.26"/>
+  <xacro:property name="base_width"   value="0.11"/>
+  <xacro:property name="base_height"  value="0.017"/>
   <!-- base_link -->
   <link name="base_link">
@@ -23,8 +23,8 @@
     </collision>
     <inertial>
-      <mass value="1.0"/>
-      <inertia ixx="0.01" ixy="0.0" ixz="0.0"
-               iyy="0.01" iyz="0.0"
-               izz="0.02"/>
+      <mass value="0.5"/>
+      <inertia ixx="0.000517" ixy="0.0"    ixz="0.0"
+               iyy="0.00283"  iyz="0.0"
+               izz="0.00332"/>
     </inertial>
   </link>
@@ -48,8 +48,8 @@
       </collision>
       <inertial>
-        <mass value="0.1"/>
-        <inertia ixx="0.001" ixy="0.0" ixz="0.0"
-                 iyy="0.001" iyz="0.0"
-                 izz="0.001"/>
+        <mass value="0.025"/>
+        <inertia ixx="9.0e-06"  ixy="0.0"    ixz="0.0"
+                 iyy="9.0e-06"  iyz="0.0"
+                 izz="1.53e-05"/>
       </inertial>
     </link>
@@ -74,24 +74,43 @@
                x="${-0.3 * base_length}"
                y="${-base_width / 2}" />
-  <!-- Gazebo 差速驱动插件 -->
+  <!-- ros2_control 硬件 + 关节接口声明 -->
+  <ros2_control name="diff_car_system" type="system">
+    <hardware>
+      <!-- 使用 Gazebo 提供的虚拟硬件 -->
+      <plugin>gazebo_ros2_control/GazeboSystem</plugin>
+    </hardware>
+    <!-- 每个轮子关节都声明 velocity 接口 -->
+    <joint name="left_front_wheel_joint">
+      <command_interface name="velocity"/>
+      <state_interface name="position"/>
+      <state_interface name="velocity"/>
+    </joint>
+    <joint name="right_front_wheel_joint">
+      <command_interface name="velocity"/>
+      <state_interface name="position"/>
+      <state_interface name="velocity"/>
+    </joint>
+    <joint name="left_behind_wheel_joint">
+      <command_interface name="velocity"/>
+      <state_interface name="position"/>
+      <state_interface name="velocity"/>
+    </joint>
+    <joint name="right_behind_wheel_joint">
+      <command_interface name="velocity"/>
+      <state_interface name="position"/>
+      <state_interface name="velocity"/>
+    </joint>
+  </ros2_control>
+  <!-- Gazebo 里加载 ros2_control 插件 -->
   <gazebo>
-    <plugin name="diff_drive" filename="libgazebo_ros_diff_drive.so">
-      <ros>
-        <namespace>/</namespace>
-        <!-- 不做重映射，直接用 /cmd_vel -->
-        <remapping>cmd_vel:=cmd_vel</remapping>
-        <remapping>odom:=odom</remapping>
-      </ros>
-      <!-- 先只用前轮两个 joint，名字必须和上面的 joint 一模一样 -->
-      <left_joint>left_front_wheel_joint</left_joint>
-      <right_joint>right_front_wheel_joint</right_joint>
-      <wheel_separation>${base_width}</wheel_separation>
-      <wheel_diameter>${2 * wheel_radius}</wheel_diameter>
-      <update_rate>50</update_rate>
-      <max_wheel_torque>5.0</max_wheel_torque>
-      <max_wheel_acceleration>3.0</max_wheel_acceleration>
-      <command_timeout>1.0</command_timeout>
-      <publish_tf>true</publish_tf>
-      <odometry_source>0</odometry_source>
+    <plugin filename="libgazebo_ros2_control.so" name="gazebo_ros2_control">
+      <!-- 告诉 gazebo_ros2_control 用哪个硬件插件（和上面 <ros2_control> 对应） -->
+      <robot_sim_type>gazebo_ros2_control/GazeboSystem</robot_sim_type>
+      <!-- 告诉它 robot_description 在哪个参数里、在哪个节点 -->
+      <robot_param>robot_description</robot_param>
+      <robot_param_node>robot_state_publisher</robot_param_node>
+      <!-- 告诉它 ros2_control 的配置 YAML 放在哪 -->
+      <robot_namespace>/diff_car</robot_namespace>
+      <parameters>$(find botlab_diff_description)/config/diff_car_ros2_control.yaml</parameters>
     </plugin>
   </gazebo>
