Commit message: diff dyn car complete

File: src/diff_dyn_car/urdf/diff_dyn_car.urdf.xacro (robot description, xacro)
@@ -30,8 +30,32 @@
   </link>
   <!-- 轮子宏 -->
+  <!-- 轮子宏：带简易“悬挂”的版本 -->
   <xacro:macro name="wheel" params="name x y">
+    <!-- 悬挂连杆：在 base_link 和 轮子 中间插一节 -->
+    <link name="${name}_susp">
+      <inertial>
+        <mass value="0.01"/>
+        <inertia ixx="1e-5" ixy="0.0" ixz="0.0"
+                 iyy="1e-5" iyz="0.0"
+                 izz="1e-5"/>
+      </inertial>
+    </link>
+    <!-- 悬挂关节：允许沿 z 方向上下走一小段（模拟压缩） -->
+    <joint name="${name}_susp_joint" type="prismatic">
+      <parent link="base_link"/>
+      <child  link="${name}_susp"/>
+      <!-- 位置还是用你之前的 x,y,z -->
+      <origin xyz="${x} ${y} -${base_height/2}" rpy="0 0 0"/>
+      <!-- z 轴方向：上下弹跳 -->
+      <axis xyz="0 0 1"/>
+      <!-- 悬挂行程：最多向下压 2 cm -->
+      <limit lower="-0.02" upper="0.0" effort="200.0" velocity="1.0"/>
+      <!-- 悬挂刚度 + 阻尼：可以再按手感调 -->
+      <dynamics spring_stiffness="1500.0" damping="50.0"/>
+    </joint>
+    <!-- 真正的轮子本体（和你之前一样） -->
     <link name="${name}">
       <visual>
-        <origin rpy="1.5708 0 0"/>
+        <origin rpy="1.57079632679 0 0"/>
         <geometry>
           <cylinder radius="${wheel_radius}" length="${wheel_width}"/>
@@ -42,5 +66,5 @@
       </visual>
       <collision>
-        <origin rpy="1.5708 0 0"/>
+        <origin rpy="1.57079632679 0 0"/>
         <geometry>
           <cylinder radius="${wheel_radius}" length="${wheel_width}"/>
@@ -48,10 +72,18 @@
         <surface>
           <contact>
-            <ode/>
+            <ode>
+              <!-- 略微可压入地面，避免太硬 -->
+              <kp>5e4</kp>
+              <kd>2.0</kd>
+              <min_depth>0.001</min_depth>
+            </ode>
           </contact>
           <friction>
             <ode>
-              <mu>0.7</mu>
-              <mu2>0.2</mu2>
+              <!-- 仍然保留你之前设置的摩擦和滑移 -->
+              <mu>0.8</mu>
+              <mu2>0.8</mu2>
+              <slip1>0.2</slip1>   <!-- 纵向滑移 -->
+              <slip2>0.2</slip2>   <!-- 横向滑移 -->
             </ode>
           </friction>
@@ -65,9 +97,13 @@
       </inertial>
     </link>
+    <!-- 保持原来的旋转关节名字：${name}_joint（给 ros2_control 用） -->
     <joint name="${name}_joint" type="continuous">
-      <parent link="base_link"/>
-      <child link="${name}"/>
-      <origin xyz="${x} ${y} -${base_height/2}" rpy="0 0 0"/>
+      <!-- 注意：现在是挂在 悬挂连杆 上 -->
+      <parent link="${name}_susp"/>
+      <child  link="${name}"/>
+      <origin xyz="0 0 0" rpy="0 0 0"/>
       <axis xyz="0 1 0"/>
+      <limit effort="5.0" velocity="100.0"/>
+      <dynamics damping="0.01" friction="0.1"/>
     </joint>
   </xacro:macro>
@@ -94,4 +130,5 @@
       <state_interface name="position"/>
       <state_interface name="velocity"/>
+      <state_interface name="effort"/>
     </joint>
     <joint name="right_front_wheel_joint">
@@ -99,4 +136,5 @@
       <state_interface name="position"/>
       <state_interface name="velocity"/>
+      <state_interface name="effort"/>
     </joint>
     <joint name="left_behind_wheel_joint">
@@ -104,4 +142,5 @@
       <state_interface name="position"/>
       <state_interface name="velocity"/>
+      <state_interface name="effort"/>
     </joint>
     <joint name="right_behind_wheel_joint">
@@ -109,4 +148,5 @@
       <state_interface name="position"/>
       <state_interface name="velocity"/>
+      <state_interface name="effort"/>
     </joint>
   </ros2_control>

Commit message: complete xbox control and change mu

File: src/diff_dyn_car/urdf/diff_dyn_car.urdf.xacro (robot description, xacro)
@@ -7,14 +7,6 @@
   <xacro:property name="base_width"   value="0.11"/>
   <xacro:property name="base_height"  value="0.017"/>
-  <!-- base_link -->
+  <!-- base_link：只做物理，不画外观 -->
   <link name="base_link">
-    <visual>
-      <geometry>
-        <box size="${base_length} ${base_width} ${base_height}"/>
-      </geometry>
-      <material name="blue">
-        <color rgba="0.1 0.3 0.9 1.0"/>
-      </material>
-    </visual>
     <collision>
       <geometry>
@@ -29,4 +21,33 @@
     </inertial>
   </link>
+  <!-- 前半段底盘：+x，车头 -->
+  <link name="base_front_link">
+    <visual>
+      <geometry>
+        <!-- 长度一半 -->
+        <box size="${base_length/2} ${base_width} ${base_height}"/>
+      </geometry>
+    </visual>
+  </link>
+  <joint name="base_front_joint" type="fixed">
+    <parent link="base_link"/>
+    <child  link="base_front_link"/>
+    <!-- 挂在 +x 方向 1/4 处 -->
+    <origin xyz="${base_length/4} 0 0" rpy="0 0 0"/>
+  </joint>
+  <!-- 后半段底盘：-x，车尾 -->
+  <link name="base_back_link">
+    <visual>
+      <geometry>
+        <box size="${base_length/2} ${base_width} ${base_height}"/>
+      </geometry>
+    </visual>
+  </link>
+  <joint name="base_back_joint" type="fixed">
+    <parent link="base_link"/>
+    <child  link="base_back_link"/>
+    <!-- 挂在 -x 方向 1/4 处 -->
+    <origin xyz="${-base_length/4} 0 0" rpy="0 0 0"/>
+  </joint>
   <!-- 轮子宏 -->
   <!-- 轮子宏：带简易“悬挂”的版本 -->
@@ -82,6 +103,6 @@
             <ode>
               <!-- 仍然保留你之前设置的摩擦和滑移 -->
-              <mu>0.8</mu>
-              <mu2>0.8</mu2>
+              <mu>1</mu>
+              <mu2>0.5</mu2>
               <slip1>0.2</slip1>   <!-- 纵向滑移 -->
               <slip2>0.2</slip2>   <!-- 横向滑移 -->
@@ -162,3 +183,23 @@
     </plugin>
   </gazebo>
+  <!-- 轮子黑色 -->
+  <gazebo reference="left_front_wheel">
+    <material>Gazebo/Black</material>
+  </gazebo>
+  <gazebo reference="right_front_wheel">
+    <material>Gazebo/Black</material>
+  </gazebo>
+  <gazebo reference="left_behind_wheel">
+    <material>Gazebo/Black</material>
+  </gazebo>
+  <gazebo reference="right_behind_wheel">
+    <material>Gazebo/Black</material>
+  </gazebo>
+  <!-- 车身：前半黄、后半蓝 -->
+  <gazebo reference="base_front_link">
+    <material>Gazebo/Yellow</material>
+  </gazebo>
+  <gazebo reference="base_back_link">
+    <material>Gazebo/Blue</material>
+  </gazebo>
 </robot>
